Commit message: add wheel position to comunication protocal

File: TEST/ROS/src/arduino_hardware_interface/test_file/test_arduino.urdf (robot description, URDF)
Before this commit: robot test_arduino_robot, 4 links, 3 joints
Links:
- removed link servo_link
- added link servo1_link
Joints:
- removed joint servo_joint
- added joint servo1_joint: type revolute, parent base_link, child servo1_link, axis 0 0 1, limit lower=-3.14 upper=3.14 effort=10 velocity=10
