Commit message: ROBOT01 NAV2 real hardware

File: ROBOT01/ROS/src/my_robot_description/urdf/mecanum_robot.urdf.xacro (robot description, xacro)
@@ -184,8 +184,8 @@
             <hardware>
                 <plugin>arduino_hardware_interface/ArduinoHardwareInterface</plugin>
-                <param name="serial_port">/dev/ttyUSB0</param>
+                <param name="serial_port">/dev/ttyNANO_L</param>
                 <param name="baudrate">115200</param>
             </hardware>
-            <joint name="front_left_wheel_joint">
+            <joint name="rear_left_wheel_joint">
                 <command_interface name="velocity"/>
                 <state_interface name="position"/>
@@ -193,5 +193,5 @@
                 <param name="direction_multiplier">1</param>
             </joint>
-            <joint name="rear_left_wheel_joint">
+            <joint name="front_left_wheel_joint">
                 <command_interface name="velocity"/>
                 <state_interface name="position"/>
@@ -228,5 +228,5 @@
                 <param name="baudrate">115200</param>
             </hardware>
-            <joint name="front_right_wheel_joint">
+            <joint name="rear_right_wheel_joint">
                 <command_interface name="velocity"/>
                 <state_interface name="position"/>
@@ -234,5 +234,5 @@
                 <param name="direction_multiplier">-1</param>
             </joint>
-            <joint name="rear_right_wheel_joint">
+            <joint name="front_right_wheel_joint">
                 <command_interface name="velocity"/>
                 <state_interface name="position"/>

Commit message: my_robot_vision init

File: ROBOT01/ROS/src/my_robot_description/urdf/mecanum_robot.urdf.xacro (robot description, xacro)
@@ -16,4 +16,15 @@
     <xacro:property name="lidar_mass"       value="0.2"/>
     <xacro:property name="lidar_x_offset"   value="0.0"/>
+    <!-- Raspberry Pi Camera Module 2 dimensions (metres). -->
+    <xacro:property name="camera_width" value="0.025"/>
+    <xacro:property name="camera_height" value="0.024"/>
+    <xacro:property name="camera_depth" value="0.009"/>
+    <xacro:property name="camera_board_depth" value="0.0016"/>
+    <xacro:property name="camera_lens_housing_depth" value="0.005"/>
+    <xacro:property name="camera_lens_housing_size" value="0.010"/>
+    <xacro:property name="camera_lens_radius" value="0.004"/>
+    <xacro:property name="camera_lens_depth" value="0.004"/>
+    <xacro:property name="camera_mass" value="0.01"/>
+    <xacro:property name="camera_update_rate" value="30"/>
     <xacro:property name="wheel_pos_x" value="${(chassis_length / 2.0) - wheel_inset_x}"/>
     <xacro:property name="wheel_pos_y" value="${(chassis_width / 2.0) + wheel_inset_y}"/>
@@ -125,4 +136,47 @@
         <child link="laser_frame"/>
         <origin xyz="${lidar_x_offset} 0 ${(chassis_height/2.0) + (lidar_height/2.0)}" rpy="0 0 0"/>
+    </joint>
+    <!-- CAMERA: +X points forward on the chassis.  The optical frame follows
+         REP 103: +Z forward, +X right, +Y down. -->
+    <link name="camera_link">
+        <!-- The board is centred on camera_link; +X is the viewing direction. -->
+        <visual>
+            <origin xyz="${-(camera_depth - camera_board_depth) / 2.0} 0 0" rpy="0 0 0"/>
+            <geometry>
+                <box size="${camera_board_depth} ${camera_width} ${camera_height}"/>
+            </geometry>
+            <material name="camera_board_green"><color rgba="0.08 0.35 0.10 1.0"/></material>
+        </visual>
+        <visual>
+            <origin xyz="${(camera_depth - camera_lens_housing_depth) / 2.0 - camera_lens_depth} 0 0" rpy="0 0 0"/>
+            <geometry>
+                <box size="${camera_lens_housing_depth} ${camera_lens_housing_size} ${camera_lens_housing_size}"/>
+            </geometry>
+            <material name="camera_lens_housing_black"><color rgba="0.04 0.04 0.04 1.0"/></material>
+        </visual>
+        <visual>
+            <origin xyz="${(camera_depth - camera_lens_depth) / 2.0} 0 0" rpy="0 ${pi / 2.0} 0"/>
+            <geometry>
+                <cylinder radius="${camera_lens_radius}" length="${camera_lens_depth}"/>
+            </geometry>
+            <material name="camera_lens_black"><color rgba="0.02 0.02 0.02 1.0"/></material>
+        </visual>
+        <collision>
+            <geometry>
+                <box size="${camera_depth} ${camera_width} ${camera_height}"/>
+            </geometry>
+        </collision>
+        <xacro:inertial_box mass="${camera_mass}" x="${camera_depth}" y="${camera_width}" z="${camera_height}"/>
+    </link>
+    <joint name="camera_joint" type="fixed">
+        <parent link="chassis"/>
+        <child link="camera_link"/>
+        <origin xyz="${(chassis_length / 2.0) + (camera_depth / 2.0)} 0 0.08" rpy="0 0 0"/>
+    </joint>
+    <link name="camera_optical_frame"/>
+    <joint name="camera_optical_joint" type="fixed">
+        <parent link="camera_link"/>
+        <child link="camera_optical_frame"/>
+        <origin xyz="0 0 0" rpy="${-pi/2} 0 ${-pi/2}"/>
     </joint>
     <!-- SENSOR LINKS FOR ROS2_CONTROL -->
@@ -323,4 +377,29 @@
             </sensor>
         </gazebo>
+        <!-- Gazebo camera rays use the camera-link convention (+X forward).
+             Messages are labelled with the ROS optical frame. -->
+        <gazebo reference="camera_link">
+            <sensor name="front_camera" type="camera">
+                <pose>0 0 0 0 0 0</pose>
+                <always_on>true</always_on>
+                <update_rate>${camera_update_rate}</update_rate>
+                <visualize>true</visualize>
+                <topic>/camera/image_raw</topic>
+                <gz_frame_id>camera_optical_frame</gz_frame_id>
+                <camera>
+                    <horizontal_fov>1.0856</horizontal_fov>
+                    <image>
+                        <width>640</width>
+                        <height>480</height>
+                        <format>R8G8B8</format>
+                    </image>
+                    <clip>
+                        <near>0.05</near>
+                        <far>20.0</far>
+                    </clip>
+                    <camera_info_topic>/camera/camera_info</camera_info_topic>
+                </camera>
+            </sensor>
+        </gazebo>
     </xacro:if>
 </robot>

Commit message: update nav2 sim

File: ROBOT01/ROS/src/my_robot_description/urdf/mecanum_robot.urdf.xacro (robot description, xacro)
@@ -5,8 +5,8 @@
     <xacro:property name="chassis_width"  value="0.30"/>
     <xacro:property name="chassis_height" value="0.05"/>
-    <xacro:property name="chassis_mass"   value="15.0"/>
+    <xacro:property name="chassis_mass"   value="0.5"/>
     <xacro:property name="wheel_radius"   value="0.0325"/>
     <xacro:property name="wheel_thickness" value="0.03"/>
-    <xacro:property name="wheel_mass"     value="1.5"/>
+    <xacro:property name="wheel_mass"     value="0.1"/>
     <xacro:property name="ground_clearance" value="0.05"/>
     <xacro:property name="wheel_inset_x" value="0.045"/>
@@ -101,5 +101,6 @@
             <child link="${prefix}_wheel"/>
             <origin xyz="${x_reflect * wheel_pos_x} ${y_reflect * wheel_pos_y} ${wheel_pos_z}" rpy="0 0 0"/>
-            <axis xyz="0 ${z_axis_reflect} 0"/>
+            <!-- <axis xyz="0 ${z_axis_reflect} 0"/> -->
+            <axis xyz="0 1 0"/>
         </joint>
         <gazebo reference="${prefix}_wheel">
@@ -321,5 +322,5 @@
     <xacro:if value="$(arg use_sim)">
         <gazebo>
-            <plugin filename="gz-sim-mecanum-drive-system" name="gz::sim::systems::MecanumDrive">
+            <!-- <plugin filename="gz-sim-mecanum-drive-system" name="gz::sim::systems::MecanumDrive">
                 <front_left_joint>front_left_wheel_joint</front_left_joint>
                 <front_right_joint>front_right_wheel_joint</front_right_joint>
@@ -335,4 +336,11 @@
                 <frame_id>odom</frame_id>
                 <child_frame_id>base_link</child_frame_id>
+            </plugin> -->
+            <plugin filename="gz-sim-odometry-publisher-system" name="gz::sim::systems::OdometryPublisher">
+                <odom_frame>odom</odom_frame>
+                <robot_base_frame>base_link</robot_base_frame>
+                <odom_topic>/odom</odom_topic>
+                <tf_topic>/tf</tf_topic>
+                <odom_publish_frequency>50</odom_publish_frequency>
             </plugin>
             <plugin filename="gz-sim-velocity-control-system" name="gz::sim::systems::VelocityControl">
@@ -352,5 +360,5 @@
                 <always_on>true</always_on>
                 <update_rate>${lidar_update_rate}</update_rate>
-                <visualize>true</visualize>
+                <visualize>false</visualize>
                 <topic>/scan</topic>
                 <gz_frame_id>laser_frame</gz_frame_id>
@@ -384,5 +392,5 @@
                 <always_on>true</always_on>
                 <update_rate>${camera_update_rate}</update_rate>
-                <visualize>true</visualize>
+                <visualize>false</visualize>
                 <topic>/camera/image_raw</topic>
                 <gz_frame_id>camera_optical_frame</gz_frame_id>

Commit message: update urdf to small robot

File: ROBOT01/ROS/src/my_robot_description/urdf/mecanum_robot.urdf.xacro (robot description, xacro)
@@ -2,12 +2,12 @@
 <robot xmlns:xacro="http://www.ros.org/wiki/xacro" name="mecanum_robot">
     <!-- chassis properties -->
-    <xacro:property name="chassis_length" value="0.45"/>
+    <xacro:property name="chassis_length" value="0.35"/>
     <xacro:property name="chassis_width"  value="0.30"/>
-    <xacro:property name="chassis_height" value="0.05"/>
+    <xacro:property name="chassis_height" value="0.005"/>
     <xacro:property name="chassis_mass"   value="0.5"/>
     <xacro:property name="wheel_radius"   value="0.0325"/>
     <xacro:property name="wheel_thickness" value="0.03"/>
     <xacro:property name="wheel_mass"     value="0.1"/>
-    <xacro:property name="ground_clearance" value="0.05"/>
+    <xacro:property name="ground_clearance" value="0.04"/>
     <xacro:property name="wheel_inset_x" value="0.045"/>
     <xacro:property name="wheel_inset_y" value="0.015"/>
@@ -15,5 +15,5 @@
     <xacro:property name="lidar_height"     value="0.05"/>
     <xacro:property name="lidar_mass"       value="0.2"/>
-    <xacro:property name="lidar_x_offset"   value="0.0"/>
+    <xacro:property name="lidar_x_offset"   value="-0.10"/>
     <!-- Raspberry Pi Camera Module 2 dimensions (metres). -->
     <xacro:property name="camera_width" value="0.025"/>

Commit message: update nav2 sim param

File: ROBOT01/ROS/src/my_robot_description/urdf/mecanum_robot.urdf.xacro (robot description, xacro)
@@ -21,8 +21,4 @@
     <xacro:property name="camera_depth" value="0.009"/>
     <xacro:property name="camera_board_depth" value="0.0016"/>
-    <xacro:property name="camera_lens_housing_depth" value="0.005"/>
-    <xacro:property name="camera_lens_housing_size" value="0.010"/>
-    <xacro:property name="camera_lens_radius" value="0.004"/>
-    <xacro:property name="camera_lens_depth" value="0.004"/>
     <xacro:property name="camera_mass" value="0.01"/>
     <xacro:property name="camera_update_rate" value="30"/>
@@ -149,18 +145,4 @@
             <material name="camera_board_green"><color rgba="0.08 0.35 0.10 1.0"/></material>
         </visual>
-        <visual>
-            <origin xyz="${(camera_depth - camera_lens_housing_depth) / 2.0 - camera_lens_depth} 0 0" rpy="0 0 0"/>
-            <geometry>
-                <box size="${camera_lens_housing_depth} ${camera_lens_housing_size} ${camera_lens_housing_size}"/>
-            </geometry>
-            <material name="camera_lens_housing_black"><color rgba="0.04 0.04 0.04 1.0"/></material>
-        </visual>
-        <visual>
-            <origin xyz="${(camera_depth - camera_lens_depth) / 2.0} 0 0" rpy="0 ${pi / 2.0} 0"/>
-            <geometry>
-                <cylinder radius="${camera_lens_radius}" length="${camera_lens_depth}"/>
-            </geometry>
-            <material name="camera_lens_black"><color rgba="0.02 0.02 0.02 1.0"/></material>
-        </visual>
         <collision>
             <geometry>
@@ -179,5 +161,5 @@
         <parent link="camera_link"/>
         <child link="camera_optical_frame"/>
-        <origin xyz="0 0 0" rpy="${-pi/2} 0 ${-pi/2}"/>
+        <origin xyz="0.0 0 0" rpy="${-pi/2} 0 ${-pi/2}"/>
     </joint>
     <!-- SENSOR LINKS FOR ROS2_CONTROL -->

Commit message: update urdf

File: ROBOT01/ROS/src/my_robot_description/urdf/mecanum_robot.urdf.xacro (robot description, xacro)
@@ -13,7 +13,8 @@
     <xacro:property name="wheel_inset_y" value="0.015"/>
     <xacro:property name="lidar_radius"     value="0.035"/>
-    <xacro:property name="lidar_height"     value="0.05"/>
+    <xacro:property name="lidar_height"     value="0.025"/>
     <xacro:property name="lidar_mass"       value="0.2"/>
-    <xacro:property name="lidar_x_offset"   value="-0.10"/>
+    <xacro:property name="lidar_x_offset"   value="-0.075"/>
+    <xacro:property name="lidar_z_offset"   value="0.21"/>
     <!-- Raspberry Pi Camera Module 2 dimensions (metres). -->
     <xacro:property name="camera_width" value="0.025"/>
@@ -23,4 +24,7 @@
     <xacro:property name="camera_mass" value="0.01"/>
     <xacro:property name="camera_update_rate" value="30"/>
+    <xacro:property name="camera_x_offset"   value="0.01"/>
+    <xacro:property name="camera_y_offset"   value="${ (chassis_width/2.0) - 0.01}"/>
+    <xacro:property name="camera_z_offset"   value="0.025"/>
     <xacro:property name="wheel_pos_x" value="${(chassis_length / 2.0) - wheel_inset_x}"/>
     <xacro:property name="wheel_pos_y" value="${(chassis_width / 2.0) + wheel_inset_y}"/>
@@ -132,5 +136,5 @@
         <parent link="chassis"/>
         <child link="laser_frame"/>
-        <origin xyz="${lidar_x_offset} 0 ${(chassis_height/2.0) + (lidar_height/2.0)}" rpy="0 0 0"/>
+        <origin xyz="${lidar_x_offset} 0 ${(chassis_height/2.0) + (lidar_height/2.0) + (lidar_z_offset)}" rpy="0 0 0"/>
     </joint>
     <!-- CAMERA: +X points forward on the chassis.  The optical frame follows
@@ -155,5 +159,5 @@
         <parent link="chassis"/>
         <child link="camera_link"/>
-        <origin xyz="${(chassis_length / 2.0) + (camera_depth / 2.0)} 0 0.08" rpy="0 0 0"/>
+        <origin xyz="${(camera_depth / 2.0) + camera_x_offset} ${camera_y_offset} ${chassis_height/2.0 + camera_height/2.0 + camera_z_offset}" rpy="0 0 1.5708"/>
     </joint>
     <link name="camera_optical_frame"/>

Commit message: small robot hardware first run

File: ROBOT01/ROS/src/my_robot_description/urdf/mecanum_robot.urdf.xacro (robot description, xacro)
@@ -16,4 +16,5 @@
     <xacro:property name="lidar_mass"       value="0.2"/>
     <xacro:property name="lidar_x_offset"   value="-0.075"/>
+    <!-- <xacro:property name="lidar_x_offset"   value="0.0"/> -->
     <xacro:property name="lidar_z_offset"   value="0.21"/>
     <!-- Raspberry Pi Camera Module 2 dimensions (metres). -->

Commit message: robot localization: init

File: ROBOT01/ROS/src/my_robot_description/urdf/mecanum_robot.urdf.xacro (robot description, xacro)
@@ -41,4 +41,9 @@
     <xacro:property name="wheelbase"        value="${wheel_pos_x * 2.0}"/>
     <xacro:property name="wheel_separation" value="${wheel_pos_y * 2.0}"/>
+    <xacro:property name="imu_sensor_L_x_offset" value="-0.075"/>
+    <xacro:property name="imu_sensor_L_y_offset" value="0.085"/>
+    <xacro:property name="imu_sensor_R_x_offset" value="-0.075"/>
+    <xacro:property name="imu_sensor_R_y_offset" value="0.09"/>
+    <xacro:property name="imu_sensor_z_offset" value="0.2"/>
     <!-- Sim Toggle -->
     <xacro:arg name="use_sim" default="false" />
@@ -169,15 +174,15 @@
     </joint>
     <!-- SENSOR LINKS FOR ROS2_CONTROL -->
-    <link name="imu_sensor_1"/>
-    <joint name="imu_1_joint" type="fixed">
-        <parent link="chassis"/>
-        <child link="imu_sensor_1"/>
-        <origin xyz="0 0 0" rpy="0 0 0"/>
-    </joint>
-    <link name="imu_sensor_2"/>
-    <joint name="imu_2_joint" type="fixed">
-        <parent link="chassis"/>
-        <child link="imu_sensor_2"/>
-        <origin xyz="0 0 0" rpy="0 0 0"/>
+    <link name="imu_sensor_L"/>
+    <joint name="imu_L_joint" type="fixed">
+        <parent link="chassis"/>
+        <child link="imu_sensor_L"/>
+        <origin xyz="${imu_sensor_L_x_offset} ${imu_sensor_L_y_offset} ${imu_sensor_z_offset}" rpy="0 0 0"/>
+    </joint>
+    <link name="imu_sensor_R"/>
+    <joint name="imu_R_joint" type="fixed">
+        <parent link="chassis"/>
+        <child link="imu_sensor_R"/>
+        <origin xyz="${imu_sensor_R_x_offset} ${imu_sensor_R_y_offset} ${imu_sensor_z_offset}" rpy="0 0 0"/>
     </joint>
     <link name="ir_sensor_1"/>
@@ -245,5 +250,5 @@
                 <state_interface name="position"/>
             </joint>
-            <sensor name="imu_sensor_1">
+            <sensor name="imu_sensor_L">
                 <state_interface name="orientation.x"/>
                 <state_interface name="orientation.y"/>
@@ -286,5 +291,5 @@
                 <state_interface name="position"/>
             </joint>
-            <sensor name="imu_sensor_2">
+            <sensor name="imu_sensor_R">
                 <state_interface name="orientation.x"/>
                 <state_interface name="orientation.y"/>
@@ -327,6 +332,7 @@
                 <odom_frame>odom</odom_frame>
                 <robot_base_frame>base_link</robot_base_frame>
-                <odom_topic>/odom</odom_topic>
-                <tf_topic>/tf</tf_topic>
+                <odom_topic>/odometry/wheel</odom_topic>
+                <!-- The EKF, rather than raw simulation, owns odom to base_link. -->
+                <tf_topic>/odometry/wheel_tf</tf_topic>
                 <odom_publish_frequency>50</odom_publish_frequency>
             </plugin>
@@ -341,4 +347,44 @@
                 <joint>rear_right_wheel_joint</joint>
             </plugin>
+        </gazebo>
+        <gazebo reference="imu_sensor_L">
+            <sensor name="imu_sensor_L_sim" type="imu">
+                <always_on>true</always_on>
+                <update_rate>50</update_rate>
+                <topic>/imu_sensor_L_broadcaster/imu</topic>
+                <gz_frame_id>imu_sensor_L</gz_frame_id>
+                <imu>
+                    <angular_velocity>
+                        <x><noise type="gaussian"><mean>0.0</mean><stddev>0.002</stddev></noise></x>
+                        <y><noise type="gaussian"><mean>0.0</mean><stddev>0.002</stddev></noise></y>
+                        <z><noise type="gaussian"><mean>0.0</mean><stddev>0.002</stddev></noise></z>
+                    </angular_velocity>
+                    <linear_acceleration>
+                        <x><noise type="gaussian"><mean>0.0</mean><stddev>0.02</stddev></noise></x>
+                        <y><noise type="gaussian"><mean>0.0</mean><stddev>0.02</stddev></noise></y>
+                        <z><noise type="gaussian"><mean>0.0</mean><stddev>0.02</stddev></noise></z>
+                    </linear_acceleration>
+                </imu>
+            </sensor>
+        </gazebo>
+        <gazebo reference="imu_sensor_R">
+            <sensor name="imu_sensor_R_sim" type="imu">
+                <always_on>true</always_on>
+                <update_rate>50</update_rate>
+                <topic>/imu_sensor_R_broadcaster/imu</topic>
+                <gz_frame_id>imu_sensor_R</gz_frame_id>
+                <imu>
+                    <angular_velocity>
+                        <x><noise type="gaussian"><mean>0.0</mean><stddev>0.002</stddev></noise></x>
+                        <y><noise type="gaussian"><mean>0.0</mean><stddev>0.002</stddev></noise></y>
+                        <z><noise type="gaussian"><mean>0.0</mean><stddev>0.002</stddev></noise></z>
+                    </angular_velocity>
+                    <linear_acceleration>
+                        <x><noise type="gaussian"><mean>0.0</mean><stddev>0.02</stddev></noise></x>
+                        <y><noise type="gaussian"><mean>0.0</mean><stddev>0.02</stddev></noise></y>
+                        <z><noise type="gaussian"><mean>0.0</mean><stddev>0.02</stddev></noise></z>
+                    </linear_acceleration>
+                </imu>
+            </sensor>
         </gazebo>
         <gazebo reference="laser_frame">

Commit message: update real hardware nav2_params

File: ROBOT01/ROS/src/my_robot_description/urdf/mecanum_robot.urdf.xacro (robot description, xacro)
@@ -10,4 +10,9 @@
     <xacro:property name="wheel_mass"     value="0.1"/>
     <xacro:property name="ground_clearance" value="0.04"/>
+    <!-- Temporary gripper collision footprint. -->
+    <xacro:property name="gripper_box_length" value="0.18"/>
+    <xacro:property name="gripper_box_width" value="0.25"/>
+    <xacro:property name="gripper_box_height" value="0.005"/>
+    <xacro:property name="gripper_box_mass" value="0.05"/>
     <xacro:property name="wheel_inset_x" value="0.045"/>
     <xacro:property name="wheel_inset_y" value="0.015"/>
@@ -86,4 +91,31 @@
         <origin xyz="0 0 ${chassis_pos_z}" rpy="0 0 0"/>
     </joint>
+    <!-- Placeholder gripper collision box. Its 25 cm side is parallel to the
+         robot width (Y), and its 18 cm side extends forward along +X. -->
+    <link name="gripper_collision_box">
+        <visual>
+            <geometry>
+                <box size="${gripper_box_length} ${gripper_box_width} ${gripper_box_height}"/>
+            </geometry>
+            <material name="gripper_orange">
+                <color rgba="0.9 0.4 0.05 0.7"/>
+            </material>
+        </visual>
+        <collision>
+            <geometry>
+                <box size="${gripper_box_length} ${gripper_box_width} ${gripper_box_height}"/>
+            </geometry>
+        </collision>
+        <xacro:inertial_box
+            mass="${gripper_box_mass}"
+            x="${gripper_box_length}"
+            y="${gripper_box_width}"
+            z="${gripper_box_height}"/>
+    </link>
+    <joint name="gripper_collision_box_joint" type="fixed">
+        <parent link="chassis"/>
+        <child link="gripper_collision_box"/>
+        <origin xyz="${(chassis_length + gripper_box_length) / 2.0} 0 0" rpy="0 0 0"/>
+    </joint>
     <xacro:macro name="mecanum_wheel" params="prefix x_reflect y_reflect z_axis_reflect">
         <link name="${prefix}_wheel">
