Commit message: add gripper box in urdf

File: ROBOT01/ROS/src/my_robot_description/urdf/mecanum_robot.urdf.xacro (robot description, xacro)
@@ -5,5 +5,5 @@
     <xacro:property name="chassis_width"  value="0.30"/>
     <xacro:property name="chassis_height" value="0.005"/>
-    <xacro:property name="chassis_mass"   value="0.5"/>
+    <xacro:property name="chassis_mass"   value="1.5"/>
     <xacro:property name="wheel_radius"   value="0.0325"/>
     <xacro:property name="wheel_thickness" value="0.03"/>
@@ -13,6 +13,6 @@
     <xacro:property name="gripper_box_length" value="0.18"/>
     <xacro:property name="gripper_box_width" value="0.25"/>
-    <xacro:property name="gripper_box_height" value="0.005"/>
-    <xacro:property name="gripper_box_mass" value="0.05"/>
+    <xacro:property name="gripper_box_height" value="0.02"/>
+    <xacro:property name="gripper_box_mass" value="0.25"/>
     <xacro:property name="wheel_inset_x" value="0.045"/>
     <xacro:property name="wheel_inset_y" value="0.015"/>
@@ -46,8 +46,8 @@
     <xacro:property name="wheelbase"        value="${wheel_pos_x * 2.0}"/>
     <xacro:property name="wheel_separation" value="${wheel_pos_y * 2.0}"/>
-    <xacro:property name="imu_sensor_L_x_offset" value="-0.075"/>
-    <xacro:property name="imu_sensor_L_y_offset" value="0.085"/>
-    <xacro:property name="imu_sensor_R_x_offset" value="-0.075"/>
-    <xacro:property name="imu_sensor_R_y_offset" value="0.09"/>
+    <xacro:property name="imu_sensor_L_x_offset" value="-0.105"/>
+    <xacro:property name="imu_sensor_L_y_offset" value="0.080"/>
+    <xacro:property name="imu_sensor_R_x_offset" value="-0.105"/>
+    <xacro:property name="imu_sensor_R_y_offset" value="-0.090"/>
     <xacro:property name="imu_sensor_z_offset" value="0.2"/>
     <!-- Sim Toggle -->

Commit message: parce tracking: hardware test, vision: frame optimize

File: ROBOT01/ROS/src/my_robot_description/urdf/mecanum_robot.urdf.xacro (robot description, xacro)
@@ -197,5 +197,6 @@
         <parent link="chassis"/>
         <child link="camera_link"/>
-        <origin xyz="${(camera_depth / 2.0) + camera_x_offset} ${camera_y_offset} ${chassis_height/2.0 + camera_height/2.0 + camera_z_offset}" rpy="0 0 1.5708"/>
+        <!-- The physical camera is upside down: roll pi about its viewing axis. -->
+        <origin xyz="${(camera_depth / 2.0) + camera_x_offset} ${camera_y_offset} ${chassis_height/2.0 + camera_height/2.0 + camera_z_offset}" rpy="0 0 ${pi/2}"/>
     </joint>
     <link name="camera_optical_frame"/>

Commit message: update camera pose

File: ROBOT01/ROS/src/my_robot_description/urdf/mecanum_robot.urdf.xacro (robot description, xacro)
@@ -30,7 +30,7 @@
     <xacro:property name="camera_mass" value="0.01"/>
     <xacro:property name="camera_update_rate" value="30"/>
-    <xacro:property name="camera_x_offset"   value="0.01"/>
-    <xacro:property name="camera_y_offset"   value="${ (chassis_width/2.0) - 0.01}"/>
-    <xacro:property name="camera_z_offset"   value="0.025"/>
+    <xacro:property name="camera_x_offset"   value="0.0205"/>
+    <xacro:property name="camera_y_offset"   value="${ (chassis_width/2.0) - 0.002}"/>
+    <xacro:property name="camera_z_offset"   value="0.01855"/>
     <xacro:property name="wheel_pos_x" value="${(chassis_length / 2.0) - wheel_inset_x}"/>
     <xacro:property name="wheel_pos_y" value="${(chassis_width / 2.0) + wheel_inset_y}"/>

Commit message: robot gripper: init

File: ROBOT01/ROS/src/my_robot_description/urdf/mecanum_robot.urdf.xacro (robot description, xacro)
@@ -243,17 +243,17 @@
         <origin xyz="-0.2 -0.1 0" rpy="0 0 0"/>
     </joint>
-    <!-- SERVO 1 (Front) -->
-    <link name="servo_1_link"/>
-    <joint name="servo_1_joint" type="continuous">
-        <parent link="chassis"/>
-        <child link="servo_1_link"/>
+    <!-- LEFT SERVO (Front) -->
+    <link name="servo_L_link"/>
+    <joint name="servo_L_joint" type="continuous">
+        <parent link="chassis"/>
+        <child link="servo_L_link"/>
         <origin xyz="0.2 0.0 0.1" rpy="0 0 0"/>
         <axis xyz="0 0 1"/>
     </joint>
-    <!-- SERVO 2 (Rear) -->
-    <link name="servo_2_link"/>
-    <joint name="servo_2_joint" type="continuous">
-        <parent link="chassis"/>
-        <child link="servo_2_link"/>
+    <!-- RIGHT SERVO (Rear) -->
+    <link name="servo_R_link"/>
+    <joint name="servo_R_joint" type="continuous">
+        <parent link="chassis"/>
+        <child link="servo_R_link"/>
         <origin xyz="-0.2 0.0 0.1" rpy="0 0 0"/>
         <axis xyz="0 0 1"/>
@@ -279,5 +279,5 @@
                 <param name="direction_multiplier">1</param>
             </joint>
-            <joint name="servo_1_joint">
+            <joint name="servo_L_joint">
                 <command_interface name="position"/>
                 <state_interface name="position"/>
@@ -320,5 +320,5 @@
                 <param name="direction_multiplier">-1</param>
             </joint>
-            <joint name="servo_2_joint">
+            <joint name="servo_R_joint">
                 <command_interface name="position"/>
                 <state_interface name="position"/>

Commit message: gray image tuning

File: ROBOT01/ROS/src/my_robot_description/urdf/mecanum_robot.urdf.xacro (robot description, xacro)
@@ -29,5 +29,5 @@
     <xacro:property name="camera_board_depth" value="0.0016"/>
     <xacro:property name="camera_mass" value="0.01"/>
-    <xacro:property name="camera_update_rate" value="30"/>
+    <xacro:property name="camera_update_rate" value="10"/>
     <xacro:property name="camera_x_offset"   value="0.0205"/>
     <xacro:property name="camera_y_offset"   value="${ (chassis_width/2.0) - 0.002}"/>
@@ -468,5 +468,5 @@
                         <width>640</width>
                         <height>480</height>
-                        <format>R8G8B8</format>
+                        <format>L8</format>
                     </image>
                     <clip>
